File: flightsim-joystick-hardware.sch (KiCad schematic (older format))
At the start: 18 parts, among them J1 USB_OTG, J2 Conn_01x02, J3 Conn_01x02, P1 CONN_02X03, U1 ATMEGA328P-AU, Y1 12MHz

Commit message: add 2 more ADC connectors
Parts:
- added J4: Conn_01x02, TerminalBlock:TerminalBlock_bornier-2_P5.08mm, symbol Connector_Generic:Conn_01x02
- R5: footprint Resistors_ThroughHole:R_Axial_DIN0204_L3.6mm_D1.6mm_P7.62mm_Horizontal -> Resistor_SMD:R_0805_2012Metric
- U1: symbol MCU_Atmel_ATMEGA:ATMEGA328P-AU -> MCU_Atmel_AVR:ATmega328P-AU
Connections:
- net Z_Pos: now reaches U1.25 (PC2)
- net Z_Pos: now also J4.1 (Pin_1)
- net W_Pos: now reaches U1.26 (PC3)
- net W_Pos: now also J4.2 (Pin_2)
- no-connect marks 15 -> 13
Other:
- moved on the sheet: C1, C4, C5, P1, R4, Y1
